File: Altaris_MCU.kicad_pcb (KiCad board)
At the start: 4 copper layers, 101.1 x 69.8 mm, 67 parts, among them J1 Screw_Terminal_01x02, J11 Screw_Terminal_01x02, J12 Screw_Terminal_01x02, J13 Screw_Terminal_01x02, J14 Screw_Terminal_01x02, J2 Conn_01x04_Pin, J3 Screw_Terminal_01x02, J4 Screw_Terminal_01x02, J5 Conn_01x04_Pin, J6 Conn_01x04_Pin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

Commit message: minor edits to layout and schematic
Routing:
- net +3.3V_b: track 54.1 -> 57.0 mm, vias 16 -> 17
Changed lines of the file:
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@@
+	)
+	(segment
+		(start 161 107.84)
+		(end 162.66 107.84)
+		(width 0.2)
+		(layer "F.Cu")
+		(net 2)
 	)
 	(segment
@@
 	)
 	(segment
+		(start 162.66 107.84)
+		(end 163.5 107)
+		(width 0.2)
+		(layer "F.Cu")
+		(net 2)
+	)
+	(segment
 		(start 157.575 123.375)
 		(end 157.9 123.7)
@@
 		(size 0.6)
 		(drill 0.3)
+		(layers "F.Cu" "B.Cu")
+		(net 2)
+	)
+	(via
+		(at 163.5 107)
+		(size 0.6)
+		(drill 0.3)

Commit message: fixed an error with netting
Routing:
- net MISO: vias 8 -> 6
- net GND: vias 501 -> 504
- net CLK: vias 11 -> 10
Changed lines of the file:
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@@
 	)
 	(via
+		(at 196.1 112.8)
+		(size 0.6)
+		(drill 0.3)
+		(layers "F.Cu" "B.Cu")
+		(free yes)
+		(net 1)
+	)
+	(via
 		(at 117.2 77.9)
 		(size 0.6)
@@
 	)
 	(via
+		(at 196.1 108.8)
+		(size 0.6)
+		(drill 0.3)
+		(layers "F.Cu" "B.Cu")
+		(free yes)
+		(net 1)
+	)
+	(via
 		(at 194.1 126.8)
 		(size 0.6)
@@
 	)
 	(via
+		(at 196.1 110.8)
+		(size 0.6)
+		(drill 0.3)
+		(layers "F.Cu" "B.Cu")
+		(free yes)
+		(net 1)
+	)
+	(via
 		(at 198.1 120.8)
 		(size 0.6)
@@
 	)
 	(via
-		(at 196.1 108.8)
-		(size 0.6)
-		(drill 0.3)
-		(layers "F.Cu" "B.Cu")
-		(net 20)
-	)
-	(via
 		(at 155.6 75.38)
 		(size 0.6)
@@
 	)
 	(via
-		(at 196.1 112.8)
-		(size 0.6)
-		(drill 0.3)
-		(layers "F.Cu" "B.Cu")
-		(net 30)
-	)
-	(via
 		(at 141.1 89.8)
 		(size 0.6)
@@
 		(size 0.6)
 		(drill 0.3)
-		(layers "F.Cu" "B.Cu")
-		(net 30)
-	)
-	(via
-		(at 196.1 110.8)
-		(size 0.6)
-		(drill 0.3)
